File: hardware/PiADC2.kicad_pcb (KiCad board)
At the start: 2 copper layers, 0 parts

Commit message: Completed version 1
Parts:
- added BT1: Battery_Cell, BH401:BH401, F.Cu at (165.1, 94.0)
- added C1: C_Small, Capacitor_SMD:C_0603_1608Metric, F.Cu at (149.2, 82.1)
- added C2: C_Small, Capacitor_SMD:C_0603_1608Metric, F.Cu at (149.2, 85.6)
- added C3: 0.1uF, Capacitor_SMD:C_0603_1608Metric, F.Cu at (127.6, 109.2)
- added C4: 0.1uF, Capacitor_SMD:C_0603_1608Metric, F.Cu at (126.4, 94.0)
- added C5: 0.1uF, Capacitor_SMD:C_0603_1608Metric, F.Cu at (146.1, 88.3)
- added C6: 0.1uF, Capacitor_SMD:C_0603_1608Metric, F.Cu at (132.7, 94.1)
- added C7: 0.1uF, Capacitor_SMD:C_0603_1608Metric, F.Cu at (148.6, 104.9)
- added C8: 0.1uF, Capacitor_SMD:C_0603_1608Metric, F.Cu at (166.4, 106.5)
- added D1: BAT54S, Package_TO_SOT_SMD:SOT-23, F.Cu at (122.6, 95.9)
- added D10: LED2, LED_SMD:LED_0603_1608Metric, F.Cu at (146.1, 92.1)
- added D2: BAT54S, Package_TO_SOT_SMD:SOT-23, F.Cu at (127.6, 103.9)
- added D3: BAT54S, Package_TO_SOT_SMD:SOT-23, F.Cu at (122.6, 111.1)
- added D4: BAT54S, Package_TO_SOT_SMD:SOT-23, F.Cu at (127.6, 119.1)
- added D5: BAT54S, Package_TO_SOT_SMD:SOT-23, F.Cu at (127.6, 98.1)
- added D6: BAT54S, Package_TO_SOT_SMD:SOT-23, F.Cu at (122.6, 106.0)
- added D7: BAT54S, Package_TO_SOT_SMD:SOT-23, F.Cu at (127.6, 113.3)
- added D8: BAT54S, Package_TO_SOT_SMD:SOT-23, F.Cu at (122.6, 121.3)
- added D9: LED1, LED_SMD:LED_0603_1608Metric, F.Cu at (146.1, 98.4)
- added J1: Pi GPIO, raspberry_pi:pi_b_hat, F.Cu at (139.7, 77.5)
- added J2: ADCIN1, Connector_JST:JST_PUD_B10B-PUDSS_2x05_P2.00mm_Vertical, F.Cu at (111.7, 103.7)
- added J3: ADCIN2, Connector_JST:JST_PUD_B10B-PUDSS_2x05_P2.00mm_Vertical, F.Cu at (111.7, 118.9)
- added J4: ISO_IN_1, JST-XA:B04B-XASK-1(LF)(SN), F.Cu at (141.0, 126.4)
- added J5: ISO_IN_2, JST-XA:B04B-XASK-1(LF)(SN), F.Cu at (155.6, 126.4)
- added J6: I2C_OUT, Connector_PinHeader_2.54mm:PinHeader_1x04_P2.54mm_Vertical, F.Cu at (126.4, 126.4)
- added JP1: ENABLE_CAL, Connector_PinHeader_1.27mm:PinHeader_1x02_P1.27mm_Vertical, F.Cu at (130.8, 90.2)
- added LOGO1: SYM_Magnet_Small, CapConiX_Logos:CapConiX_Logo_10_7, F.Cu at (111.8, 86.4)
- added LOGO2: SYM_Magnet_Small, Symbol:OSHW-Logo_5.7x6mm_SilkScreen, F.Cu at (168.3, 118.7)
- added R1: 1K, Resistor_SMD:R_0603_1608Metric, F.Cu at (118.7, 97.8)
- added R10: 1K, Resistor_SMD:R_0603_1608Metric, F.Cu at (118.7, 119.4)
- added R11: 10K, Resistor_SMD:R_0603_1608Metric, F.Cu at (122.6, 90.8)
- added R12: 10K, Resistor_SMD:R_0603_1608Metric, F.Cu at (118.7, 90.8)
- added R13: 10K, Resistor_SMD:R_0603_1608Metric, F.Cu at (126.4, 86.4)
- added R14: 10K, Resistor_SMD:R_0603_1608Metric, F.Cu at (138.9, 104.1)
- added R15: 10K, Resistor_SMD:R_0603_1608Metric, F.Cu at (143.0, 104.1)
- added R16: 10K, Resistor_SMD:R_0603_1608Metric, F.Cu at (153.5, 104.1)
- added R17: 10K, Resistor_SMD:R_0603_1608Metric, F.Cu at (157.6, 104.1)
- added R18: 10K, Resistor_SMD:R_0603_1608Metric, F.Cu at (159.4, 118.7)
- added R19: 10K, Resistor_SMD:R_0603_1608Metric, F.Cu at (156.8, 118.7)
- added R2: 1K, Resistor_SMD:R_0603_1608Metric, F.Cu at (118.7, 99.7)
- added R20: 10K, Resistor_SMD:R_0603_1608Metric, F.Cu at (154.3, 118.7)
- added R21: 10K, Resistor_SMD:R_0603_1608Metric, F.Cu at (151.8, 118.7)
- added R22: 10K, Resistor_SMD:R_0603_1608Metric, F.Cu at (144.8, 118.7)
- added R23: 10K, Resistor_SMD:R_0603_1608Metric, F.Cu at (142.2, 118.7)
- added R24: 10K, Resistor_SMD:R_0603_1608Metric, F.Cu at (139.7, 118.7)
- added R25: 10K, Resistor_SMD:R_0603_1608Metric, F.Cu at (137.2, 118.7)
- added R26: 470, Resistor_SMD:R_0603_1608Metric, F.Cu at (146.1, 96.5)
- added R27: 470, Resistor_SMD:R_0603_1608Metric, F.Cu at (146.1, 94.0)
- added R28: 10K, Resistor_SMD:R_0603_1608Metric, F.Cu at (164.5, 103.5)
- added R29: 10K, Resistor_SMD:R_0603_1608Metric, F.Cu at (162.6, 103.5)
- added R3: 1K, Resistor_SMD:R_0603_1608Metric, F.Cu at (118.7, 102.2)
- added R4: 1K, Resistor_SMD:R_0603_1608Metric, F.Cu at (118.7, 104.1)
- added R5: 10K, Resistor_SMD:R_0603_1608Metric, F.Cu at (122.6, 81.9)
- added R6: 10K, Resistor_SMD:R_0603_1608Metric, F.Cu at (118.7, 81.9)
- added R7: 1K, Resistor_SMD:R_0603_1608Metric, F.Cu at (118.7, 113.0)
- added R8: 1K, Resistor_SMD:R_0603_1608Metric, F.Cu at (118.7, 114.9)
- added R9: 1K, Resistor_SMD:R_0603_1608Metric, F.Cu at (118.7, 117.5)
- added SW1: SW_Push, Button_Switch_SMD:SW_SPST_TL3305A, F.Cu at (153.0, 92.1)
- added SW2: SW_Push, Button_Switch_SMD:SW_SPST_TL3305A, F.Cu at (153.0, 98.4)
- added U1: ADS1115IDGS, Package_SO:TSSOP-10_3x3mm_P0.5mm, F.Cu at (123.8, 101.0)
- added U2: TCA9517, Package_SO:MSOP-8_3x3mm_P0.65mm, F.Cu at (120.7, 86.4)
- added U3: ADS1115IDGS, Package_SO:TSSOP-10_3x3mm_P0.5mm, F.Cu at (123.8, 116.2)
- added U4: 24LC16, Package_SO:SO-8_3.9x4.9mm_P1.27mm, F.Cu at (131.4, 85.1)
- added U5: MCP79401-I_SN, Package_SO:SO-8_3.9x4.9mm_P1.27mm, F.Cu at (154.3, 85.1)
- added U6: MCP23008T-E_SS, Package_SO:SSOP-20_5.3x7.2mm_P0.65mm, F.Cu at (138.4, 95.2)
- added U7: HCPL2631M, Package_DIP:DIP-8_W7.62mm_LongPads, F.Cu at (137.2, 114.9)
- added U8: HCPL2631M, Package_DIP:DIP-8_W7.62mm_LongPads, F.Cu at (151.8, 114.9)
- added Y1: Crystal, Crystal:Crystal_DS26_D2.0mm_L6.0mm_Horizontal_1EP_style2, F.Cu at (147.1, 82.9)
Routing:
- net +3V3: track 0.00 -> 217.6 mm, vias 0 -> 6
- net +5V: track 0.00 -> 156.8 mm, vias 0 -> 9
- net I2C_SDA_3V3: track 0.00 -> 59.4 mm, vias 0 -> 3
- net I2C_SCL_3V3: track 0.00 -> 57.9 mm, vias 0 -> 3
- net GND: track 0.00 -> 53.6 mm, vias 0 -> 4
- net I2C_SCL_5V: track 0.00 -> 48.7 mm, vias 0 -> 3
- net I2C_SDA_5V: track 0.00 -> 48.2 mm, vias 0 -> 3
- net Net-(R28-Pad2): track 0.00 -> 36.7 mm
- net Net-(R29-Pad2): track 0.00 -> 26.9 mm
- net Net-(R17-Pad1): track 0.00 -> 25.8 mm
- net Net-(R16-Pad1): track 0.00 -> 23.9 mm
- net Net-(BT1-Pad1): track 0.00 -> 16.5 mm, vias 0 -> 1
- net Net-(R15-Pad1): track 0.00 -> 12.5 mm
- net Net-(D4-Pad3): track 0.00 -> 11.0 mm
- net Net-(D2-Pad3): track 0.00 -> 11.0 mm
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- added copper zone on B.Cu, net GND
- added copper zone on F.Cu, net GND
Other:
- board outline added: 65 x 56 mm
- board text added: "2020/01"
- board text added: "FOR TESTING ONLY OPEN SOURCE HARDWARE RELEASED UNDER CERN OHL v1.2"
- board text added: "PiADC2 v1 - CapConiX LLC - capconix.com"
- board text added: "PiADC2 v1 CapConiX LLC capconix.com"
